File: attenuator.sch (KiCad schematic (older format))
At the start: 37 parts, among them J1 Conn_01x03_Male, J2 Conn_01x03_Male, J3 Conn_01x02_Male, J4 Conn_01x04_Male, J5 Conn_01x02_Male, K1 G5V-2, K2 G5V-2, K3 G5V-2, K4 G5V-2, K5 G5V-2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

Commit message: change schema and working on pcb
Parts:
- removed J4: Conn_01x04_Male, Connectors_Molex:Molex_KK-6410-04_04x2.54mm_Straight, symbol Connector:Conn_01x04_Male
- removed J5: Conn_01x02_Male, Connectors_Molex:Molex_KK-6410-02_02x2.54mm_Straight, symbol Connector:Conn_01x02_Male
- added J4: Conn_01x05_Male, Connector_IDC:IDC-Header_2x05_P2.54mm_Horizontal, symbol Connector:Conn_01x05_Male
- J1, J2: footprint Connectors_Molex:Molex_KK-6410-03_03x2.54mm_Straight -> Connector_Molex:Molex_KK-254_AE-6410-03A_1x03_P2.54mm_Vertical
- J3: footprint Connectors_Molex:Molex_KK-6410-02_02x2.54mm_Straight -> Connector_Molex:Molex_KK-254_AE-6410-02A_1x02_P2.54mm_Vertical
- K1: footprint Relays_THT:Relay_DPDT_Omron_G5V-2 -> Relay_THT:Relay_DPDT_Omron_G5V-2
- R1, R10, R11, R12, R13, R14, R15, R16, R17, R18, R19, R2, R20, R21, R22, R23, R24, R3, R4, R5, R6, R7, R8, R9: footprint Resistors_THT:R_Axial_DIN0207_L6.3mm_D2.5mm_P5.08mm_Vertical -> Resistor_THT:R_Axial_DIN0309_L9.0mm_D3.2mm_P12.70mm_Horizontal
- U1, U2: footprint Housings_DIP:DIP-16_W7.62mm -> Package_DIP:DIP-16_W7.62mm
Connections:
- net labels removed: +5V
- wire segments 185 -> 183
